Commit message: checking if any files are missing while uploading

File: robot_arm_urdf/urdf/robot_arm_urdf.urdf (robot description, URDF)
Before this commit: robot robot_arm_urdf, 9 links, 8 joints
Links:
- link extrusion: geometry collision mesh filename=package://robot_arm_urdf/meshes/item_37003_profile-5-20x20-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 scale=0.001 0.001 0.001; visual mesh filename=package://robot_arm_urdf/meshes/item_37003_profile-5-20x20-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
Joints:
- joint Fixed_extrusion_frame: origin xyz=0.13 -0.1465 0.175 rpy=1.57 0 0 -> xyz=0.13 -0.1465 0 rpy=0 0 0
